Commit message: goalPost and ball added

File: goal_post.urdf (robot description, URDF)
Before this commit: robot GoalPost, 1 links, 0 joints
Links:
- removed link Post
- added link back_side, mass .0; collision mesh filename=goal_post/goal_post_back_col.stl scale=0.1 0.1 0.1; visual mesh filename=goal_post/goal_post_back_col.stl scale=0.1 0.1 0.1
- added link bottom_side, mass .0; collision mesh filename=goal_post/goal_post_cover_col.stl scale=0.1 0.1 0.1; visual mesh filename=goal_post/goal_post_cover_col.stl scale=0.1 0.1 0.1
- added link left_side, mass .0; collision mesh filename=goal_post/goal_post_side_col.stl scale=0.1 0.1 0.1; visual mesh filename=goal_post/goal_post_side_col.stl scale=0.1 0.1 0.1
- added link right_side, mass .0; collision mesh filename=goal_post/goal_post_side_col.stl scale=0.1 0.1 0.1; visual mesh filename=goal_post/goal_post_side_col.stl scale=0.1 0.1 0.1
- added link top_side, mass .0; collision mesh filename=goal_post/goal_post_cover_col.stl scale=0.1 0.1 0.1; visual mesh filename=goal_post/goal_post_cover_col.stl scale=0.1 0.1 0.1
Joints:
- added joint link_bottom_side_back: type fixed, parent back_side, child bottom_side, origin xyz=1.0 0 0 rpy=0 0 0
- added joint link_left_side_back: type fixed, parent back_side, child right_side, origin xyz=1.0 0 0 rpy=0 0 0
- added joint link_right_side_back: type fixed, parent back_side, child left_side, origin xyz=1.0 0 0 rpy=0 0 0
- added joint link_top_side_back: type fixed, parent back_side, child top_side, origin xyz=1.0 0 0 rpy=0 0 0
